File: hardware/src/PCB/FPV_drone/Analog_video.kicad_sch (KiCad schematic)
At the start: 1 part, among them IC7 AT7456E

Commit message: Update: schem almost finish
Parts:
- removed IC7: AT7456E, SOP65P640X120-29N, symbol lib:AT7456E
- added C12, C13: 12pF, Capacitor_THT:C_Disc_D3.0mm_W2.0mm_P2.50mm, symbol PCM_SL_Devices:Capacitor_NP
- added C48, C51, C52, C53: 100nF, Capacitor_THT:C_Disc_D3.0mm_W2.0mm_P2.50mm, symbol PCM_SL_Devices:Capacitor_NP
- added C49, C50: 22uF, Capacitor_THT:C_Disc_D3.0mm_W2.0mm_P2.50mm, symbol PCM_SL_Devices:Capacitor_NP
- added J3: Conn_01x06, PCM_SparkFun-Connector:JST_1x06_P1.0mm_Horizontal_SMD, symbol PCM_SparkFun-Connector:Conn_01x06_JST_P1.0mm_Horizontal_SMD
- added J5, J6: JST_1mm_4, PCM_SparkFun-Connector:JST_1x04_P1.0mm_Horizontal_SMD, symbol PCM_SparkFun-Connector:Conn_01x04_JST_P1.0mm_Horizontal_SMD
- added R36: 1kΩ, symbol Device:R
- added R37, R38: 75Ω, symbol Device:R
- added R39: 10kΩ, symbol Device:R
- added U2: AT7456ELAH_C42388749, symbol lib:AT7456ELAH_C42388749
- added Y2: ABM3B-27.000MHZ-10-B-1-U-T, ABM3B, symbol lib:ABM3B-8.000MHZ-10-D1G-T
Connections:
- new net: C49.1, U2.16 (VOUT)
- new net: C49.2, C50.2, R38.2
- new net: C52.2, U2.13 (VIN)
- new net: R36.2, U2.9 (RESET#)
- new net: C50.1, U2.15 (SAG)
- new net +10V: J3.6
- new net +3.3V: C48.1, C51.2, C53.2, R36.1, R39.1, U2.12 (AVDD), U2.14 (PVDD), U2.2 (DVDD)
- new net DJI_RX: J3.3
- new net DJI_SBUS: J3.1
- new net DJI_TX: J3.4
- new net Earth: C12.2, C13.1, J3.2, J3.5, R37.2, Y2.2 (GND_1), Y2.4 (GND_2)
- new net GNDA: C53.1, U2.10 (AGND), U2.17 (EP1), U2.18 (EP2)
- new net GNDD: C48.2, U2.1 (DGND)
- new net GNDPWR: C51.1, U2.11 (PGND)
- new net ISC_IN: C13.2, U2.3 (CLKIN), Y2.1 (XTAL_1)
- new net ISC_OUT: C12.1, U2.4 (XFB), Y2.3 (XTAL_2)
- new net OSD_CS: R39.2, U2.5 (CS#)
- new net OSD_MISO: U2.8 (SDOUT)
- new net OSD_MOSI: U2.6 (SDIN)
- new net OSD_SCK: U2.7 (SCLK)
- new net VIDEO_IN: C52.1, R37.1
- new net VIDEO_OUT: R38.1
Other:
- note added: "Analog VTX OSD - AT7456ELAH"
- note added: "Analog VTX OSD - Crystal 0scillator - 27MHz +/-10ppm 50Ω 10pF"
- note added: "CL_reel = (C1*C2)/(C1+C2) + C_stray = (12*12)/(12+12) + ~3pF = 6 + 3 = 9-10 pF"
- note added: "Connectors"

Commit message: Update: bit changes
Changed lines of the file:
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@@
 	(wire
 		(pts
-			(xy 156.21 44.45) (xy 157.48 44.45)
+			(xy 156.21 44.45) (xy 160.02 44.45)
 		)
 		(stroke
@@
 	(wire
 		(pts
-			(xy 156.21 36.83) (xy 157.48 36.83)
+			(xy 156.21 36.83) (xy 160.02 36.83)
 		)
 		(stroke
@@
 	(wire
 		(pts
-			(xy 156.21 34.29) (xy 157.48 34.29)
+			(xy 156.21 34.29) (xy 160.02 34.29)
 		)
 		(stroke
@@
 	(symbol
 		(lib_id "power:Earth")
-		(at 157.48 44.45 90)
+		(at 160.02 44.45 90)
 		(unit 1)
 		(body_style 1)
@@
 		(dnp no)
 		(property "Reference" "#PWR039"
-			(at 163.83 44.45 0)
+			(at 166.37 44.45 0)
 			(hide yes)
 			(show_name no)
@@
 		)
 		(property "Value" "Earth"
-			(at 162.56 44.45 90)
+			(at 165.1 44.45 90)
 			(show_name no)
 			(do_not_autoplace no)
@@
 		)
 		(property "Footprint" ""
-			(at 157.48 44.45 0)
+			(at 160.02 44.45 0)
 			(hide yes)
 			(show_name no)
@@
 		)
 		(property "Datasheet" ""
-			(at 157.48 44.45 0)
+			(at 160.02 44.45 0)
 			(hide yes)
 			(show_name no)
@@
 		)
 		(property "Description" "Power symbol creates a global label with name \"Earth\""
-			(at 157.48 44.45 0)
+			(at 160.02 44.45 0)
 			(hide yes)
 			(show_name no)
@@
 	(symbol
 		(lib_id "power:+9V")
-		(at 157.48 34.29 270)
+		(at 160.02 34.29 270)
 		(unit 1)
 		(body_style 1)
@@
 		(dnp no)
 		(property "Reference" "#PWR0107"
-			(at 153.67 34.29 0)
+			(at 156.21 34.29 0)
 			(hide yes)
 			(show_name no)
@@
 		)
 		(property "Value" "+10V"
-			(at 160.274 34.29 90)
+			(at 162.814 34.29 90)
 			(show_name no)
 			(do_not_autoplace no)
@@
 		)
 		(property "Footprint" ""
-			(at 157.48 34.29 0)
+			(at 160.02 34.29 0)
 			(hide yes)
 			(show_name no)
@@
 		)
 		(property "Datasheet" ""
-			(at 157.48 34.29 0)
+			(at 160.02 34.29 0)
 			(hide yes)
 			(show_name no)
@@
 		)
 		(property "Description" "Power symbol creates a global label with name \"+9V\""
-			(at 157.48 34.29 0)
+			(at 160.02 34.29 0)
 			(hide yes)
 			(show_name no)
@@
 	(symbol
 		(lib_id "power:Earth")
-		(at 157.48 36.83 90)
+		(at 160.02 36.83 90)
 		(unit 1)
 		(body_style 1)
@@
 		(dnp no)
 		(property "Reference" "#PWR040"
-			(at 163.83 36.83 0)
+			(at 166.37 36.83 0)
 			(hide yes)
 			(show_name no)
@@
 		)
 		(property "Value" "Earth"
-			(at 162.56 36.83 90)
+			(at 165.1 36.83 90)
 			(show_name no)
 			(do_not_autoplace no)
@@
 		)
 		(property "Footprint" ""
-			(at 157.48 36.83 0)
+			(at 160.02 36.83 0)
 			(hide yes)
 			(show_name no)
@@
 		)
 		(property "Datasheet" ""
-			(at 157.48 36.83 0)
+			(at 160.02 36.83 0)
 			(hide yes)
 			(show_name no)
@@
 		)
 		(property "Description" "Power symbol creates a global label with name \"Earth\""
-			(at 157.48 36.83 0)
+			(at 160.02 36.83 0)
 			(hide yes)
 			(show_name no)

Commit message: update: schem finished
Parts:
- added D2: SMBJ12A, LIB:DIONM5436X261N, symbol lib:SMBJ12A
- U2: footprint (none) -> LIB:AT7456ELAH
- Y2: footprint ABM3B -> LIB:ABM3B
Connections:
- net +10V: now also J6.1, D2.1 (K)
- net Earth: now also J5.2, J6.2, D2.2 (A)
- net VIDEO_IN: now also J5.3
- net VIDEO_OUT: now also J6.3
- net +5V: now reaches J5.1
- net CAM_C: now reaches J5.4
- net IRC: now reaches J6.4
Other:
- moved on the sheet: J3, J5, J6

Commit message: Update: schem finished
Parts:
- removed D2: SMBJ12A, LIB:DIONM5436X261N, symbol lib:SMBJ12A
Other:
- moved on the sheet: R37
