File: hardware/src/PCB/FPV_drone/Power_functions.kicad_sch (KiCad schematic)
At the start: 35 parts, among them IC1 TPS2121RUXT, IC4 AP2112K-3.3TRG1, IC5 DCP3603BCMR - 500kHz, IC8 DCP3603BCMR - 500kHz, J2 Batt

Commit message: Update: schem drone
power functions almost finish... i wish
Parts:
- removed J2: Batt, symbol Connector_Generic:Conn_01x02
- added C20, C29: 1uF, Capacitor_THT:C_Disc_D3.0mm_W2.0mm_P2.50mm, symbol PCM_SL_Devices:Capacitor_NP
- added IC10: AP2112K-3.3TRG1, SOT95P285X140-5N, symbol lib:AP2112K-3.3TRG1
- added IC3: USBLC6-2SC6, SOT95P280X145-6N, symbol lib:USBLC6-2SC6
- added J1: TYPE-C-31-M-12, TYPE-C-31-M-12:HRO_TYPE-C-31-M-12, symbol lib:TYPE-C-31-M-12
- added R1, R2: 5.1kΩ, symbol Device:R
- added R27, R28: 5kΩ, symbol Device:R
- C28: value 22uF -> 100uF
Connections:
- net +5V: now also C28.1, C29.1, IC10.1 (VIN), IC10.3 (EN); no longer C16.2, C26.2, C28.2, C46.2, IC1.6 (PR1), IC1.7 (IN1), L1.2, R14.2, R18.1
- net +9V: now also L2.2
- net Earth: now also C28.2, IC1.3 (CP2), R13.1, C20.2, C29.2, IC10.2 (GND), IC3.2 (GND), J1.A1_B12 (GND), J1.B1_A12 (GND), J1.S1 (SHIELD), J1.S2 (SHIELD), J1.S3 (SHIELD), J1.S4 (SHIELD), R1.1, R2.2, R28.2; no longer C28.1
- net at C30.2, IC1.11 (SS): no longer IC1.3 (CP2), R13.1
- net at L2.1: now also IC8.6 (SW)
- net +26V renamed BATT+
- net USB_PROTECTION renamed +5V_USB
- net +5V_USB: now also IC3.5 (VBUS), J1.A4_B9 (VBUS), J1.B4_A9 (VBUS)
- new net: IC1.6 (PR1), R27.1, R28.1
- new net: J1.A5 (CC1), R1.2
- new net: J1.B5 (CC2), R2.1
- new net +3.3V_IMU2: C20.1, IC10.5 (VOUT)
- new net +5V_buck: C16.2, C26.2, C46.2, IC1.7 (IN1), L1.2, R14.2, R18.1, R27.2
- new net DN1: IC3.1 (I/O1_1), J1.A7 (DN1), J1.B7 (DN2)
- new net DP1: IC3.3 (I/O2_1), J1.A6 (DP1), J1.B6 (DP2)
- new net USB_DN: IC3.6 (I/O1_2)
- new net USB_DP: IC3.4 (I/O2_2)
- no-connect marks 2 -> 5
Other:
- moved on the sheet: C17, C18, C26, C27, C28, C30, D1, IC1, R13, R18, R19, R20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

Commit message: Update: schem almost finish
Parts:
- added C44, C45: 22uF-50V, Capacitor_THT:C_Disc_D3.0mm_W2.0mm_P2.50mm, symbol PCM_SL_Devices:Capacitor_NP
- C18: value 100nF - 50V -> 100nF-50V
- C26: value 22uF -> 100nF
- IC5, IC8: value DCP3603BCMR - 500kHz -> DCP3603ACMR - 500kHz
- R22: value 143kΩ -> 162kΩ
Connections:
- net BATT+: now also C44.1, C45.1
- net Earth: now also C44.2, C45.2
- net +9V renamed +10V
Other:
- note added: "3.3V 600mA LDO"
- note added: "36V max input - 10V 3A Buck"
- note added: "36V max input - 5V 3A Buck"
- note added: "500kHz 0.07% Ripple"
- note added: "500kHz 0.09% Ripple"
- note added: "Batt decoupling (2s - 8s)"
- note added: "Ideal diode multiplexer - 2,08A 56mΩ"
- note added: "One dedicate to a IMU"
- note added: "Power path mux between two source (here Batt and USB)"
- note added: "USB input 5V - ESD protection"
- note removed: "TVS- 12V"
- moved on the sheet: C15, C16, C17, C18, C19, C20, C21, C25, C26, C27, C28, C29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

Commit message: Update: bit changes
Other:
- note added: "A revoir peut aucun filtre juste TVS qui est a changer btw"
Changed lines of the file:
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@@
+		)
+	)
+	(text "A revoir peut aucun filtre juste TVS qui est a changer btw"
+		(exclude_from_sim no)
+		(at 81.28 23.876 0)
+		(effects
+			(font
+				(size 1.27 1.27)
+			)
 		)
 	)

Commit message: update: schem finished
Parts:
- removed C18: 100nF-50V, Capacitor_THT:C_Disc_D3.0mm_W2.0mm_P2.50mm, symbol PCM_SL_Devices:Capacitor_NP
- removed C26: 100nF, Capacitor_THT:C_Disc_D3.0mm_W2.0mm_P2.50mm, symbol PCM_SL_Devices:Capacitor_NP
- removed C27: 4.7uF, Capacitor_THT:C_Disc_D3.0mm_W2.0mm_P2.50mm, symbol PCM_SL_Devices:Capacitor_NP
- removed C38: 100nF - 50V, Capacitor_THT:C_Disc_D3.0mm_W2.0mm_P2.50mm, symbol PCM_SL_Devices:Capacitor_NP
- removed D1: SMBJ33A, DIOM5436X244N, symbol lib:SMBJ33A
- removed R28: 5kΩ, symbol Device:R
- added D1: SMBJ40A, LIB:DIOM5436X261N, symbol lib:SMBJ40A
- added D3: SMBJ6.0A-TR, LIB:SMBJ12A, symbol lib:SMBJ6.0A-TR
- C16, C25, C41, C46: value 22uF -> 22uF-25V
- C28: value 100uF -> 100nF
- C45: value 22uF-50V -> 100nF - 50V
- IC1: footprint TPS2121RUXT -> LIB:TPS2121RUXT
- IC10, IC4: footprint SOT95P285X140-5N -> LIB:SOT95P285X140-5N
- IC3: footprint SOT95P280X145-6N -> LIB:SOT95P280X145-6N
- IC5, IC8: footprint SOT95P280X125-6N -> LIB:SOT95P280X125-6N
- J1: footprint TYPE-C-31-M-12:HRO_TYPE-C-31-M-12 -> LIB:HRO_TYPE-C-31-M-12
- L1, L2: footprint 74438367100 -> LIB:74438367100
- R13: value 51.1kΩ -> 30.1kΩ
- R24, R6: value 100kΩ -> 10kΩ
Connections:
- net +5V: now also D3.1 (K)
- net BATT+: now also D1.1 (K); no longer C45.1
- net Earth: now also D1.2 (A), D3.2 (A); no longer C32.1, C45.2
- net at IC5.6 (SW), L1.1: now also C32.1
- net at IC8.6 (SW), L2.1: now also C45.1
- net at IC8.1 (BOOT): now also C45.2
Other:
- note added: "One dedicate to the IMUs"
- note removed: "A revoir peut aucun filtre juste TVS qui est a changer btw"
- note removed: "One dedicate to a IMU"
- moved on the sheet: C15, C16, C17, C25, C30, C31, C32, C41, C44, C46, IC5, IC8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

Commit message: Update: schem finished
Parts:
- removed C17: 1uF-50V, Capacitor_THT:C_Disc_D3.0mm_W2.0mm_P2.50mm, symbol PCM_SL_Devices:Capacitor_NP
- removed D3: SMBJ6.0A-TR, LIB:SMBJ12A, symbol lib:SMBJ6.0A-TR
- added C55: 22uF-50V, Capacitor_THT:C_Disc_D3.0mm_W2.0mm_P2.50mm, symbol PCM_SL_Devices:Capacitor_NP
- added D2: SMBJ12A, LIB:DIONM5436X261N, symbol lib:SMBJ12A
- added D4: SMBJ6.0A-TR, LIB:SMBJ12A, symbol lib:SMBJ6.0A-TR
- C44: value 22uF-50V -> 100nF-50V
- L1, L2: value 10uH -> 22uH
- R13: value 30.1kΩ -> 36kΩ
- R18: value 23.7kΩ -> 3.65kΩ
- R27: value 5kΩ -> 20kΩ
Connections:
- net +10V: now also D2.1 (K)
- net +5V: now also D4.1 (K)
- net +5V_buck: no longer R18.1
- net BATT+: now also C55.1
- net Earth: now also C55.2, D2.2 (A), D4.2 (A)
- net at IC1.6 (PR1), R27.1: now also R18.1
Other:
- note added: "500kHz 25,8% Ripple"
- note added: "500kHz 42,6% Ripple"
- note added: "Change for 33A"
- note added: "Ideal diode multiplexer - 2,98A 56mΩ"
- note added: "TVS overvoltage protection"
- note removed: "500kHz 0.07% Ripple"
- note removed: "500kHz 0.09% Ripple"
- note removed: "Ideal diode multiplexer - 2,08A 56mΩ"
- moved on the sheet: C44, R27
